File: hardware-6l/main.kicad_pcb (KiCad board)
At the start: 6 copper layers, 20 x 20 mm, 0 parts

Commit message: fix drc
Other:
- board size 20 x 20 mm -> 24 x 24 mm
Changed lines of the file:
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@@
+	)
+	(gr_line
+		(start 49.999999 54.000001)
+		(end 33.999999 54.000001)
+		(stroke
+			(width 0.1)
+			(type default)
+		)
+		(layer "Edge.Cuts")
+	)
+	(gr_arc
+		(start 34.000001 54.000001)
+		(mid 31.171573 52.828428)
+		(end 30 50)
+		(stroke
+			(width 0.1)
+			(type default)
+		)
+		(layer "Edge.Cuts")
 	)
 	(gr_line
@@
 		(layer "Edge.Cuts")
 	)
+	(gr_arc
+		(start 50 30)
+		(mid 52.828428 31.171573)
+		(end 54.000001 34.000001)
+		(stroke
+			(width 0.1)
+			(type default)
+		)
+		(layer "Edge.Cuts")
+	)
+	(gr_arc
+		(start 54 50)
+		(mid 52.828427 52.828428)
+		(end 49.999999 54.000001)
+		(stroke
+			(width 0.1)
+			(type default)
+		)
+		(layer "Edge.Cuts")
+	)
 	(gr_line
 		(start 29.999999 34.000001)
@@
 		(stroke
 			(width 0.1)
+			(type default)
+		)
+		(layer "Edge.Cuts")
+	)
+	(gr_line
+		(start 54 49.999999)
+		(end 54 34)
+		(stroke
+			(width 0.1)
