File: hardware/main.kicad_sch (KiCad schematic)
At the start: 0 parts

Commit message: update stack
Other:
- company: ELT -> SET!!!
Changed lines of the file:
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@@
 		(date "SET!!!")
 		(rev "VERV")
-		(company "ELT")
+		(company "SET!!!")
 		(comment 2 "SET!!!")
 		(comment 4 "SET!!!")

Commit message: Update to kicad9
Parts:
- added FID1, FID2, FID3: Fiducial, MAS_Package_std:Fiducial_1mm_Mask2mm, symbol Mechanical:Fiducial
